File: kicad/PiHat.kicad_sch (KiCad schematic)
At the start: 8 parts, among them U1 SEN0291, U2 Power_Connector, U3 DS3235, U5 Raspberry_Pi_5, U6 5V_Linear_Regulator

Commit message: Add kicad pcb
Parts:
- U3: symbol GloablCustomSymbols:ServoPinHeader -> PiHatComponents:ServoPinHeader
- U4: symbol GloablCustomSymbols:RotaryEncoderPinHeader -> PiHatComponents:RotaryEncoderPinHeader
- U5: footprint Global_Custom_Library:Pi5Hat -> pi_hat:Pi5Hat; symbol GloablCustomSymbols:Pi5-Pinout -> PiHatComponents:Pi5-Pinout
- U6: value 5V_Linear_Regulator -> UBEC DC/DC Converter; footprint pi_hat:5vVoltageRegulator -> pi_hat:UBEC 5V Step Down; symbol GloablCustomSymbols:5vVoltageRegulator -> PiHatComponents:5vVoltageRegulator
Connections:
- net +3V3 is gone; now on net +5V: U1.1 (VCC)
- net Power_Servo is gone; now on net +7.5V: U1.5 (Vin), U3.2 (Vin)
- net +5V: now also U5.2 (5V_power), U5.4 (5V_power), U6.2 (VOUT)
- net +7.5V: now also U1.7 (Vout)
- net ENCODER_A: now also U5.37 (GPIO_26); no longer U5.38 (GPIO_20)
- net ENCODER_B: now also U5.31 (GPIO_6); no longer U5.40 (GPIO_21)
- net GND: now also U5.14 (Ground), U5.20 (Ground), U5.30 (Ground), U5.34 (Ground), U5.6 (Ground)
- removed net 5V_Pi_IN: U1.7 (Vout), U5.2 (5V_power), U5.4 (5V_power), U6.2 (VOUT)
Other:
- moved on the sheet: BZ1, C1, U1, U2, U3, U4, U6
